File: test.kicad_sch (KiCad schematic)
At the start: 55 parts, among them IC1 BQ24074RGTR, IC2 USBLC6-2SC6, IC3 ESP32-S3-WROOM-1-N16, J1 UART0, J2 73100-0105, J3 73100-0105, K1 AQY210EHA, SW1 Reset, SW2 Boot, U1 USB-TYPE-C-018, U2 1043, U3 1043, U4 LD1086DT33TR, U5 LD1086DT33TR

Commit message: added dac and changed switch, gain
Parts:
- removed IC?: MCP6S91-E_MS, project_library:MCP6S91-E_MS, symbol project_library:MCP6S91-E_MS
- added C14, C15, C16, C17, C18, C19, C20, C21, C22, C23, C24, C25, C26: (no value), symbol Device:C_Small
- added IC5: (no value), project_library:MCP6S91-E_MS, symbol project_library:MCP6S91-E_MS
- added IC7: (no value), project_library:MCP4726A1T-E_CH, symbol project_library:MCP4726A1T-E_CH
- added R13, R14: (no value), symbol Device:R_Small
- added R?: (no value), Resistor_SMD:R_0805_2012Metric_Pad1.20x1.40mm_HandSolder, symbol Device:R_Small
- added U7, U8: (no value), project_library:ADC08351CILQX, symbol project_library:ADC08351CILQX{brace}slash}NOPB
- C1: renamed from C?; value 1u -> (none); footprint Capacitor_SMD:C_1206_3216Metric_Pad1.33x1.80mm_HandSolder -> (none)
- C10: renamed from C7; value 10u -> (none); footprint Capacitor_SMD:C_1206_3216Metric_Pad1.33x1.80mm_HandSolder -> (none)
- C11, C8: renamed from C?; value 10u -> (none); footprint Capacitor_SMD:C_1206_3216Metric_Pad1.33x1.80mm_HandSolder -> (none)
- C12: renamed from C9; value 10u -> (none); footprint Capacitor_SMD:C_1206_3216Metric_Pad1.33x1.80mm_HandSolder -> (none)
- C13: renamed from C10; value 10u -> (none); footprint Capacitor_SMD:C_1206_3216Metric_Pad1.33x1.80mm_HandSolder -> (none)
- C2: renamed from C1; value 1u -> (none); footprint Capacitor_SMD:C_1206_3216Metric_Pad1.33x1.80mm_HandSolder -> (none)
- C27, C28: renamed from C?; value 47n -> (none); footprint Capacitor_SMD:C_1206_3216Metric_Pad1.33x1.80mm_HandSolder -> (none)
- C29, C30: renamed from C?; value 100n -> (none)
- C3: renamed from C2; value 4u7 -> (none); footprint Capacitor_SMD:C_1206_3216Metric_Pad1.33x1.80mm_HandSolder -> (none)
- C31, C32: renamed from C?; value 5.5p-30p var -> (none); footprint project_library:JZ300 -> (none)
- C4: renamed from C3; footprint Capacitor_SMD:C_1206_3216Metric_Pad1.33x1.80mm_HandSolder -> (none)
- C5: value 22u -> (none); footprint Capacitor_SMD:C_1206_3216Metric_Pad1.33x1.80mm_HandSolder -> (none)
- C6: renamed from C4; value 4u7 -> (none); footprint Capacitor_SMD:C_1206_3216Metric_Pad1.33x1.80mm_HandSolder -> (none)
- C7: renamed from C8; value 0.1u -> (none); footprint Capacitor_SMD:C_1206_3216Metric_Pad1.33x1.80mm_HandSolder -> (none)
- C9: renamed from C6; value 10u -> (none); footprint Capacitor_SMD:C_1206_3216Metric_Pad1.33x1.80mm_HandSolder -> (none)
- D1: value LED_ValidSource -> (none); footprint LED_SMD:LED_2512_6332Metric_Pad1.52x3.35mm_HandSolder -> (none)
- D2: value LED_Charging -> (none); footprint LED_SMD:LED_2512_6332Metric_Pad1.52x3.35mm_HandSolder -> (none)
- IC1: renamed from IC?; value LC709203FQH-01TWG -> (none)
- IC2: renamed from IC1; value BQ24074RGTR -> (none)
- IC3: renamed from IC2; value USBLC6-2SC6 -> (none)
- IC4: renamed from IC3; value ESP32-S3-WROOM-1-N16 -> (none)
- J1: value UART0 -> (none); footprint Connector_PinHeader_2.54mm:PinHeader_1x04_P2.54mm_Vertical -> (none)
- J2: renamed from J3; value 73100-0105 -> (none)
- J3: renamed from J2; value 73100-0105 -> (none)
- K1: value AQY210EHA -> (none)
- K2: renamed from K?; value AQY210EHA -> (none)
- R1: renamed from R?; value 10k -> (none); footprint Resistor_SMD:R_1206_3216Metric_Pad1.30x1.75mm_HandSolder -> (none)
- R10: value 120 -> (none); footprint Resistor_SMD:R_1206_3216Metric_Pad1.30x1.75mm_HandSolder -> (none)
- R11, R12: value 470 -> (none); footprint Resistor_SMD:R_1206_3216Metric_Pad1.30x1.75mm_HandSolder -> (none)
- R15, R16: renamed from R?; value 100k -> (none); footprint Resistor_SMD:R_1206_3216Metric_Pad1.30x1.75mm_HandSolder -> (none)
- R17, R18: renamed from R?; value 910k -> (none)
- R2, R4, R8: value 5k1 -> (none); footprint Resistor_SMD:R_1206_3216Metric_Pad1.30x1.75mm_HandSolder -> (none)
- R3: value 1k -> (none); footprint Resistor_SMD:R_1206_3216Metric_Pad1.30x1.75mm_HandSolder -> (none)
- R5: value 820 -> (none); footprint Resistor_SMD:R_1206_3216Metric_Pad1.30x1.75mm_HandSolder -> (none)
- R6, R7: value 1k5 -> (none); footprint Resistor_SMD:R_1206_3216Metric_Pad1.30x1.75mm_HandSolder -> (none)
- R9: value 39 -> (none); footprint Resistor_SMD:R_1206_3216Metric_Pad1.30x1.75mm_HandSolder -> (none)
- SW1: value Reset -> (none); footprint project_library:SW_TS-1187A-B-A-B -> (none)
- SW2: value Boot -> (none); footprint project_library:SW_TS-1187A-B-A-B -> (none)
- U1: renamed from U2; value 1043 -> (none)
- U2: renamed from U3; value 1043 -> (none)
- U3: renamed from U1; value USB-TYPE-C-018 -> (none); footprint project_library:USB-TYPE-C-018 -> footprint:USB-C_SMD-TYPE-C-31-M-12
- U4: renamed from U?; value LD1086DT33TR -> (none)
- U5: renamed from U4; value LD1086DT33TR -> (none)
- U6: renamed from U5; value LD1086DT33TR -> (none)
Connections:
- net +3V3: now also C14.1, C15.1, C17.1, C18.1, IC5.8 (VDD), U7.10 (VD), U7.12 (VD), U8.10 (VD), U8.12 (VD)
- net CH1_D0: now also U7.1 (D0), U8.1 (D0)
- net CH1_D1: now also U7.2 (D1), U8.2 (D1)
- net CH1_D2: now also U7.3 (D2), U8.3 (D2)
- net CH1_D3: now also U7.4 (D3), U8.4 (D3)
- net CH1_D4: now also U7.5 (D4), U8.5 (D4)
- net CH1_D5: now also U7.6 (D5), U8.6 (D5)
- net CH1_D6: now also U7.7 (D6), U8.7 (D6)
- net CH1_D7: now also U7.8 (D7), U8.8 (D7)
- net CH1_Gnd_Sel: now also K1.1 (Anode)
- net CH2_Gnd_Sel: now also K2.1 (Anode)
- net CS_A: now also IC5.5 (~{CS})
- net GND: now also C13.1, R10.1, U6.2 (OUT), C14.2, C15.2, C16.2, C17.2, C18.2, C19.2, C20.2, C21.2, C22.2, C23.2, C24.2, C25.2, C26.2, IC5.3 (VREF), IC5.4 (VSS), IC7.2 (VSS), R13.1, R14.1, R?.2, U7.15 (PD), U7.18 (AGND), U7.19 (AGND), U7.21 (DGND), U7.22 (~{OE}), U7.23 (DGND), U8.15 (PD), U8.18 (AGND), U8.19 (AGND), U8.21 (DGND), U8.22 (~{OE}), U8.23 (DGND)
- net I2S_CLK: now also U7.11 (CLK), U8.11 (CLK)
- net MOSI: now also IC5.6 (SI)
- net PGND: no longer C13.1, R10.1, U6.2 (OUT)
- net SCL: now also IC7.5 (SCL)
- net SCLK: now also IC5.7 (SCK)
- net SDA: now also IC7.4 (SDA)
- net at C29.1, C31.2, R17.2: now also K1.3 (SW); no longer K1.1 (Anode)
- net at C27.1, C29.2, R15.1: now also K1.4 (SW); no longer K1.2 (Kathode)
- net at C28.1, C30.2, R16.1: now also K2.4 (SW); no longer K2.2 (Kathode)
- net at C30.1, C32.2, R18.2: now also K2.3 (SW); no longer K2.1 (Anode)
- net +3.3VADC renamed +3.3VA
- net +3.3VA: now also C20.1, C21.1, C22.1, C23.1, C24.1, C25.1, U7.16 (VA), U8.14 (Vref), U8.16 (VA)
- new net: K1.2 (Kathode), R13.2
- new net: C26.1, IC7.1 (VOUT)
- new net: K2.2 (Kathode), R14.2
- new net: C16.1, C19.1, IC7.3 (VDD)
- new net: IC5.1 (VOUT), R?.1
- no-connect marks 15 -> 25
Other:
- note added: "16V ? Welcher R?"
- note added: "Ax Serie bedeutet I2C-Adresse unterschiedliche bestellen"
- moved on the sheet: C27, C28, C29, C30, C31, C32, J2, J3, K1, K2, R15, R16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

Commit message: grouped footprints
Parts:
- added C25, C29: 0.1u, Capacitor_SMD:C_0805_2012Metric_Pad1.18x1.45mm_HandSolder, symbol Device:C_Small
- added C27: 10u, Capacitor_SMD:C_0805_2012Metric_Pad1.18x1.45mm_HandSolder, symbol Device:C_Small
- added D1: (no value), LED_SMD:LED_0805_2012Metric_Pad1.15x1.40mm_HandSolder, symbol Device:LED_Small
- added IC6: MCP6S91-E_MS, project_library:MCP6S91-E_MS, symbol project_library:MCP6S91-E_MS
- added IC8: MCP4726A1T-E_CH, project_library:MCP4726A1T-E_CH, symbol project_library:MCP4726A1T-E_CH
- added JP?: (no value), symbol Jumper:Jumper_3_Open
- added R1: 1k5, Resistor_SMD:R_0805_2012Metric_Pad1.20x1.40mm_HandSolder, symbol Device:R_Small
- added R12: (no value), Resistor_SMD:R_0805_2012Metric_Pad1.20x1.40mm_HandSolder, symbol Device:R_Small
- added R13: 5k, Resistor_SMD:R_0805_2012Metric_Pad1.20x1.40mm_HandSolder, symbol Device:R_Small
- added R17: 5k1, Resistor_SMD:R_0805_2012Metric_Pad1.20x1.40mm_HandSolder, symbol Device:R_Small
- C1, C2, C4: value (none) -> 1u; footprint (none) -> Capacitor_SMD:C_0805_2012Metric_Pad1.18x1.45mm_HandSolder
- C10, C11, C12, C13, C8, C9: value (none) -> 10u; footprint (none) -> Capacitor_SMD:C_0805_2012Metric_Pad1.18x1.45mm_HandSolder
- C14, C15, C7: value (none) -> 0.1u; footprint (none) -> Capacitor_SMD:C_0805_2012Metric_Pad1.18x1.45mm_HandSolder
- C16: renamed from C17; value (none) -> 10u; footprint (none) -> Capacitor_SMD:C_0805_2012Metric_Pad1.18x1.45mm_HandSolder
- C17: renamed from C18; value (none) -> 10u; footprint (none) -> Capacitor_SMD:C_0805_2012Metric_Pad1.18x1.45mm_HandSolder
- C18: renamed from C20; value (none) -> 0.1u; footprint (none) -> Capacitor_SMD:C_0805_2012Metric_Pad1.18x1.45mm_HandSolder
- C19: renamed from C21; value (none) -> 0.1u; footprint (none) -> Capacitor_SMD:C_0805_2012Metric_Pad1.18x1.45mm_HandSolder
- C20: renamed from C22; value (none) -> 0.1u; footprint (none) -> Capacitor_SMD:C_0805_2012Metric_Pad1.18x1.45mm_HandSolder
- C21: renamed from C23; value (none) -> 0.1u; footprint (none) -> Capacitor_SMD:C_0805_2012Metric_Pad1.18x1.45mm_HandSolder
- C22: renamed from C24; value (none) -> 10u; footprint (none) -> Capacitor_SMD:C_0805_2012Metric_Pad1.18x1.45mm_HandSolder
- C23: renamed from C25; value (none) -> 10u; footprint (none) -> Capacitor_SMD:C_0805_2012Metric_Pad1.18x1.45mm_HandSolder
- C24: renamed from C16; value (none) -> 0.1u; footprint (none) -> Capacitor_SMD:C_0805_2012Metric_Pad1.18x1.45mm_HandSolder
- C26: renamed from C19; value (none) -> 10u; footprint (none) -> Capacitor_SMD:C_0805_2012Metric_Pad1.18x1.45mm_HandSolder
- C28: renamed from C26; value (none) -> 0.1u; footprint (none) -> Capacitor_SMD:C_0805_2012Metric_Pad1.18x1.45mm_HandSolder
- C3, C6: value (none) -> 4u7; footprint (none) -> Capacitor_SMD:C_0805_2012Metric_Pad1.18x1.45mm_HandSolder
- C30: renamed from C27; value (none) -> 47n; footprint (none) -> Capacitor_SMD:C_0805_2012Metric_Pad1.18x1.45mm_HandSolder
- C31: renamed from C28; value (none) -> 47n; footprint (none) -> Capacitor_SMD:C_0805_2012Metric_Pad1.18x1.45mm_HandSolder
- C32: renamed from C29; value (none) -> 100n; footprint (none) -> Capacitor_SMD:C_0805_2012Metric_Pad1.18x1.45mm_HandSolder
- C33: renamed from C30; value (none) -> 100n; footprint (none) -> Capacitor_SMD:C_0805_2012Metric_Pad1.18x1.45mm_HandSolder
- C34: renamed from C31; value (none) -> 5.5p-30p var; footprint (none) -> project_library:JZ300
- C35: renamed from C32; value (none) -> 5.5p-30p var; footprint (none) -> project_library:JZ300
- C5: value (none) -> 22u; footprint (none) -> Capacitor_SMD:C_0805_2012Metric_Pad1.18x1.45mm_HandSolder
- D2: renamed from D1; value (none) -> LED_ValidSource; footprint (none) -> LED_SMD:LED_0805_2012Metric_Pad1.15x1.40mm_HandSolder
- D3: renamed from D2; value (none) -> LED_Charging; footprint (none) -> LED_SMD:LED_0805_2012Metric_Pad1.15x1.40mm_HandSolder
- IC1: value (none) -> LC709203FQH-01TWG
- IC2: value (none) -> BQ24074RGTR
- IC3: value (none) -> USBLC6-2SC6
- IC4: value (none) -> ESP32-S3-WROOM-1-N16
- IC5: value (none) -> MCP6S91-E_MS
- IC7: value (none) -> MCP4726A1T-E_CH
- J1: value (none) -> UART0; footprint (none) -> Connector_PinHeader_2.54mm:PinHeader_1x04_P2.54mm_Vertical
- J2, J3: value (none) -> 73100-0105
- K1, K2: value (none) -> AQY210EHA
- R10: renamed from R9; value (none) -> 39; footprint (none) -> Resistor_SMD:R_0805_2012Metric_Pad1.20x1.40mm_HandSolder
- R11: renamed from R10; value (none) -> 120; footprint (none) -> Resistor_SMD:R_0805_2012Metric_Pad1.20x1.40mm_HandSolder
- R14: renamed from R11; value (none) -> 470; footprint (none) -> Resistor_SMD:R_0805_2012Metric_Pad1.20x1.40mm_HandSolder
- R15: renamed from R12; value (none) -> 470; footprint (none) -> Resistor_SMD:R_0805_2012Metric_Pad1.20x1.40mm_HandSolder
- R16: renamed from R?; value (none) -> 5k1
- R18: renamed from R13; value (none) -> 1k; footprint (none) -> Resistor_SMD:R_0805_2012Metric_Pad1.20x1.40mm_HandSolder
- R19: renamed from R14; value (none) -> 1k; footprint (none) -> Resistor_SMD:R_0805_2012Metric_Pad1.20x1.40mm_HandSolder
- R2: renamed from R1; value (none) -> 10k; footprint (none) -> Resistor_SMD:R_0805_2012Metric_Pad1.20x1.40mm_HandSolder
- R20: renamed from R15; value (none) -> 100k; footprint (none) -> Resistor_SMD:R_0805_2012Metric_Pad1.20x1.40mm_HandSolder
- R21: renamed from R16; value (none) -> 100k; footprint (none) -> Resistor_SMD:R_0805_2012Metric_Pad1.20x1.40mm_HandSolder
- R22: renamed from R17; value (none) -> 910k; footprint (none) -> Resistor_SMD:R_0805_2012Metric_Pad1.20x1.40mm_HandSolder
- R23: renamed from R18; value (none) -> 910k; footprint (none) -> Resistor_SMD:R_0805_2012Metric_Pad1.20x1.40mm_HandSolder
- R3: renamed from R2; value (none) -> 5k1; footprint (none) -> Resistor_SMD:R_0805_2012Metric_Pad1.20x1.40mm_HandSolder
- R4: renamed from R3; value (none) -> 1k; footprint (none) -> Resistor_SMD:R_0805_2012Metric_Pad1.20x1.40mm_HandSolder
- R5: renamed from R4; value (none) -> 5k1; footprint (none) -> Resistor_SMD:R_0805_2012Metric_Pad1.20x1.40mm_HandSolder
- R6: renamed from R5; value (none) -> 820; footprint (none) -> Resistor_SMD:R_0805_2012Metric_Pad1.20x1.40mm_HandSolder
- R7: renamed from R6; value (none) -> 1k5; footprint (none) -> Resistor_SMD:R_0805_2012Metric_Pad1.20x1.40mm_HandSolder
- R8: renamed from R7; value (none) -> 1k5; footprint (none) -> Resistor_SMD:R_0805_2012Metric_Pad1.20x1.40mm_HandSolder
- R9: renamed from R8; value (none) -> 5k1; footprint (none) -> Resistor_SMD:R_0805_2012Metric_Pad1.20x1.40mm_HandSolder
- SW2: value (none) -> Boot; footprint (none) -> project_library:SW_TS-1187A-B-A-B
- U1, U2: value (none) -> 1043
- U3: value (none) -> USB-TYPE-C-018
- U4, U5, U6: value (none) -> LD1086DT33TR
- U7, U8: value (none) -> ADC08351CILQX/NOPB
Connections:
- net PGND is gone; now on net GND: C30.2, C31.2, J2.1, J2.2, J3.1, J3.2, R20.2, R21.2
- net +3V3: now also IC6.8 (VDD), R12.2, R13.2
- net +5V: now also JP?.3 (B)
- net Alarm: now also R1.2
- net CS_A: now also IC6.5 (~{CS})
- net GND: now also C25.2, C27.2, C29.2, D1.1 (K), IC6.3 (VREF), IC6.4 (VSS), IC8.2 (VSS), R17.2
- net MOSI: now also IC6.6 (SI)
- net RX0: no longer J1.2 (Pin_2), R14.2
- net SCL: now also IC8.5 (SCL), R12.1
- net SCLK: now also IC6.7 (SCK)
- net SDA: now also IC8.4 (SDA), R13.1
- net TX0: no longer J1.3 (Pin_3), R15.2
- net Vbat: now also JP?.1 (A); no longer C10.1, C8.1, C9.1, U4.3 (IN), U5.3 (IN), U6.3 (IN)
- net ValidUSB: no longer names the net of D2.1 (K), IC2.7 (~{PGOOD})
- new net: D1.2 (A), R1.1
- new net: C10.1, C8.1, C9.1, JP?.2 (C), U4.3 (IN), U5.3 (IN), U6.3 (IN)
- new net: C29.1, IC8.1 (VOUT)
- new net: C25.1, C27.1, IC8.3 (VDD)
- new net: IC6.1 (VOUT), R17.1
- new net RX: J1.2 (Pin_2), R14.2
- new net TX: J1.3 (Pin_3), R15.2
Other:
- moved on the sheet: C10, C11, C12, C13, C24, C26, C28, C30, C31, C32, C33, C34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

Commit message: groups new aranged
Parts:
- removed SW1: (no value), symbol Switch:SW_Push
- removed SW2: Boot, project_library:SW_TS-1187A-B-A-B, symbol Switch:SW_Push
- added SW1: (no value), symbol project_library:Button
- added SW2: (no value), project_library:SW_TS-1187A-B-A-B, symbol project_library:Button
- C1, C2, C4: value 1u -> (none); footprint Capacitor_SMD:C_0805_2012Metric_Pad1.18x1.45mm_HandSolder -> (none)
- C10, C11, C12, C13, C16, C17, C22, C23, C26, C27, C8, C9: value 10u -> (none); footprint Capacitor_SMD:C_0805_2012Metric_Pad1.18x1.45mm_HandSolder -> (none)
- C14, C15, C18, C19, C20, C21, C24, C25, C28, C29, C7: value 0.1u -> (none); footprint Capacitor_SMD:C_0805_2012Metric_Pad1.18x1.45mm_HandSolder -> (none)
- C3, C6: value 4u7 -> (none); footprint Capacitor_SMD:C_0805_2012Metric_Pad1.18x1.45mm_HandSolder -> (none)
- C30, C31: value 47n -> (none); footprint Capacitor_SMD:C_0805_2012Metric_Pad1.18x1.45mm_HandSolder -> (none)
- C32, C33: value 100n -> (none); footprint Capacitor_SMD:C_0805_2012Metric_Pad1.18x1.45mm_HandSolder -> (none)
- C34, C35: value 5.5p-30p var -> (none); footprint project_library:JZ300 -> (none)
- C5: value 22u -> (none); footprint Capacitor_SMD:C_0805_2012Metric_Pad1.18x1.45mm_HandSolder -> (none)
- D1: footprint LED_SMD:LED_0805_2012Metric_Pad1.15x1.40mm_HandSolder -> (none)
- D2: value LED_ValidSource -> (none); footprint LED_SMD:LED_0805_2012Metric_Pad1.15x1.40mm_HandSolder -> (none)
- D3: value LED_Charging -> (none); footprint LED_SMD:LED_0805_2012Metric_Pad1.15x1.40mm_HandSolder -> (none)
- IC1: value LC709203FQH-01TWG -> (none)
- IC2: value BQ24074RGTR -> (none)
- IC3: value USBLC6-2SC6 -> (none)
- IC4: value ESP32-S3-WROOM-1-N16 -> (none)
- IC5, IC6: value MCP6S91-E_MS -> (none)
- IC7, IC8: value MCP4726A1T-E_CH -> (none)
- J1: value UART0 -> (none); footprint Connector_PinHeader_2.54mm:PinHeader_1x04_P2.54mm_Vertical -> (none)
- J2, J3: value 73100-0105 -> (none)
- K1, K2: value AQY210EHA -> (none)
- R1, R7, R8: value 1k5 -> (none); footprint Resistor_SMD:R_0805_2012Metric_Pad1.20x1.40mm_HandSolder -> (none)
- R10: value 39 -> (none); footprint Resistor_SMD:R_0805_2012Metric_Pad1.20x1.40mm_HandSolder -> (none)
- R11: renamed from R12; footprint Resistor_SMD:R_0805_2012Metric_Pad1.20x1.40mm_HandSolder -> (none)
- R12: renamed from R11; value 120 -> (none); footprint Resistor_SMD:R_0805_2012Metric_Pad1.20x1.40mm_HandSolder -> (none)
- R13: value 5k -> (none); footprint Resistor_SMD:R_0805_2012Metric_Pad1.20x1.40mm_HandSolder -> (none)
- R14, R15: value 470 -> (none); footprint Resistor_SMD:R_0805_2012Metric_Pad1.20x1.40mm_HandSolder -> (none)
- R16, R17, R9: value 5k1 -> (none); footprint Resistor_SMD:R_0805_2012Metric_Pad1.20x1.40mm_HandSolder -> (none)
- R18, R19: value 1k -> (none); footprint Resistor_SMD:R_0805_2012Metric_Pad1.20x1.40mm_HandSolder -> (none)
- R2: renamed from R3; value 5k1 -> (none); footprint Resistor_SMD:R_0805_2012Metric_Pad1.20x1.40mm_HandSolder -> (none)
- R20, R21: value 100k -> (none); footprint Resistor_SMD:R_0805_2012Metric_Pad1.20x1.40mm_HandSolder -> (none)
- R22, R23: value 910k -> (none); footprint Resistor_SMD:R_0805_2012Metric_Pad1.20x1.40mm_HandSolder -> (none)
- R3: renamed from R2; value 10k -> (none); footprint Resistor_SMD:R_0805_2012Metric_Pad1.20x1.40mm_HandSolder -> (none)
- R4: renamed from R5; value 5k1 -> (none); footprint Resistor_SMD:R_0805_2012Metric_Pad1.20x1.40mm_HandSolder -> (none)
- R5: renamed from R4; value 1k -> (none); footprint Resistor_SMD:R_0805_2012Metric_Pad1.20x1.40mm_HandSolder -> (none)
- R6: value 820 -> (none); footprint Resistor_SMD:R_0805_2012Metric_Pad1.20x1.40mm_HandSolder -> (none)
- U1, U2: value 1043 -> (none)
- U3: value USB-TYPE-C-018 -> (none)
- U4, U5, U6: value LD1086DT33TR -> (none)
- U7, U8: value ADC08351CILQX/NOPB -> (none)
- gave numbers to parts that had none: 1
Connections:
- net BOOT: now also SW2.A, SW2.B
- net CH1_D0: now also IC4.11 (IO18); no longer IC4.4 (IO4), U8.1 (D0)
- net CH1_D1: now also IC4.10 (IO17); no longer IC4.5 (IO5), U8.2 (D1)
- net CH1_D2: now also IC4.9 (IO16); no longer IC4.6 (IO6), U8.3 (D2)
- net CH1_D3: now also IC4.8 (IO15); no longer IC4.7 (IO7), U8.4 (D3)
- net CH1_D4: now also IC4.7 (IO7); no longer IC4.8 (IO15), U8.5 (D4)
- net CH1_D5: now also IC4.6 (IO6); no longer IC4.9 (IO16), U8.6 (D5)
- net CH1_D6: now also IC4.5 (IO5); no longer IC4.10 (IO17), U8.7 (D6)
- net CH1_D7: now also IC4.4 (IO4); no longer IC4.11 (IO18), U8.8 (D7)
- net CH2_D0: now also IC4.25 (IO48), U8.1 (D0); no longer IC4.15 (IO3)
- net CH2_D1: now also IC4.24 (IO47), U8.2 (D1); no longer IC4.17 (IO9)
- net CH2_D2: now also IC4.23 (IO21), U8.3 (D2); no longer IC4.18 (IO10)
- net CH2_D3: now also IC4.22 (IO14), U8.4 (D3); no longer IC4.21 (IO13)
- net CH2_D4: now also IC4.21 (IO13), U8.5 (D4); no longer IC4.22 (IO14)
- net CH2_D5: now also IC4.18 (IO10), U8.6 (D5); no longer IC4.23 (IO21)
- net CH2_D6: now also IC4.17 (IO9), U8.7 (D6); no longer IC4.24 (IO47)
- net CH2_D7: now also IC4.15 (IO3), U8.8 (D7); no longer IC4.25 (IO48)
- net ENABLE: now also SW1.C, SW1.D
- net GND: now also SW1.A, SW1.B, SW2.C, SW2.D
Other:
- moved on the sheet: R2, R4, U3
