File: test.kicad_sch (KiCad schematic)
At the start: 20 parts, among them IC2 AD9288BSTZ-40, U3 ESP32-WROOM-E

Commit message: routing
Parts:
- C18: value (none) -> 10u; footprint (none) -> Capacitor_SMD:C_0603_1608Metric_Pad1.08x0.95mm_HandSolder
- C7: value (none) -> 22u; footprint (none) -> Capacitor_SMD:C_0603_1608Metric_Pad1.08x0.95mm_HandSolder
- C8: value (none) -> 0.1u; footprint (none) -> Capacitor_SMD:C_0603_1608Metric_Pad1.08x0.95mm_HandSolder
Changed lines of the file:
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@@
-    (effects (font (size 1.27 1.27)) (justify right bottom))
-  )
-  (label "IO0" (at 189.23 81.28 180)
     (effects (font (size 1.27 1.27)) (justify right bottom))
   )
@@
     (effects (font (size 1.27 1.27)) (justify right bottom))
   )
-  (label "RX" (at 189.23 76.2 180)
-    (effects (font (size 1.27 1.27)) (justify right bottom))
-  )
   (label "CH1_D2" (at 44.45 106.68 180)
     (effects (font (size 1.27 1.27)) (justify right bottom))
@@
     (effects (font (size 1.27 1.27)) (justify right bottom))
   )
-  (label "ENABLE" (at 189.23 68.58 180)
-    (effects (font (size 1.27 1.27)) (justify right bottom))
-  )
   (label "I2S_CLK" (at 259.08 99.06 0)
     (effects (font (size 1.27 1.27)) (justify left bottom))
@@
     (effects (font (size 1.27 1.27)) (justify right bottom))
   )
-  (label "TX" (at 189.23 78.74 180)
-    (effects (font (size 1.27 1.27)) (justify right bottom))
-  )
   (label "CH2_D1" (at 266.7 71.12 180)
     (effects (font (size 1.27 1.27)) (justify right bottom))
@@
   (label "CH1_D6" (at 44.45 96.52 180)
     (effects (font (size 1.27 1.27)) (justify right bottom))
+  )
+  (global_label "ENABLE" (shape input) (at 189.23 68.58 180) (fields_autoplaced)
+    (effects (font (size 1.27 1.27)) (justify right))
+    (property "Intersheet References" "${INTERSHEET_REFS}" (id 0) (at 179.8017 68.5006 0)
+      (effects (font (size 1.27 1.27)) (justify right) hide)
+    )
   )
   (global_label "Offset_CH1" (shape input) (at 259.08 93.98 0) (fields_autoplaced)
@@
     (property "Intersheet References" "${INTERSHEET_REFS}" (id 0) (at 77.3906 52.1364 90)
       (effects (font (size 1.27 1.27)) (justify left) hide)
+    )
+  )
+  (global_label "IO0" (shape input) (at 189.23 81.28 180) (fields_autoplaced)
+    (effects (font (size 1.27 1.27)) (justify right))
+    (property "Intersheet References" "${INTERSHEET_REFS}" (id 0) (at 183.6721 81.2006 0)
+      (effects (font (size 1.27 1.27)) (justify right) hide)
     )
   )
@@
     )
   )
+  (global_label "RX" (shape input) (at 189.23 76.2 180) (fields_autoplaced)
+    (effects (font (size 1.27 1.27)) (justify right))
+    (property "Intersheet References" "${INTERSHEET_REFS}" (id 0) (at 184.3374 76.1206 0)
+      (effects (font (size 1.27 1.27)) (justify right) hide)
+    )
+  )
+  (global_label "TX" (shape input) (at 189.23 78.74 180) (fields_autoplaced)
+    (effects (font (size 1.27 1.27)) (justify right))
+    (property "Intersheet References" "${INTERSHEET_REFS}" (id 0) (at 184.6398 78.6606 0)
+      (effects (font (size 1.27 1.27)) (justify right) hide)
+    )
+  )
   (global_label "Trigger_CH1" (shape input) (at 193.04 116.84 180) (fields_autoplaced)
     (effects (font (size 1.27 1.27)) (justify right))
@@
       (effects (font (size 1.27 1.27)) (justify left))
     )
-    (property "Value" "" (id 1) (at 170.18 138.4362 0)
-      (effects (font (size 1.27 1.27)) (justify left))
-    )
-    (property "Footprint" "" (id 2) (at 167.64 137.16 0)
+    (property "Value" "22u" (id 1) (at 170.18 138.4362 0)
+      (effects (font (size 1.27 1.27)) (justify left))
+    )
+    (property "Footprint" "Capacitor_SMD:C_0603_1608Metric_Pad1.08x0.95mm_HandSolder" (id 2) (at 167.64 137.16 0)
       (effects (font (size 1.27 1.27)) hide)
     )
@@
       (effects (font (size 1.27 1.27)) (justify left))
     )
-    (property "Value" "" (id 1) (at 179.07 138.4362 0)
-      (effects (font (size 1.27 1.27)) (justify left))
-    )
-    (property "Footprint" "" (id 2) (at 176.53 137.16 0)
+    (property "Value" "0.1u" (id 1) (at 179.07 138.4362 0)
+      (effects (font (size 1.27 1.27)) (justify left))
+    )
+    (property "Footprint" "Capacitor_SMD:C_0603_1608Metric_Pad1.08x0.95mm_HandSolder" (id 2) (at 176.53 137.16 0)
       (effects (font (size 1.27 1.27)) hide)
     )
@@
       (effects (font (size 1.27 1.27)) (justify left))
     )
-    (property "Value" "" (id 1) (at 111.7662 63.5 0)
-      (effects (font (size 1.27 1.27)) (justify left))
-    )
-    (property "Footprint" "" (id 2) (at 110.49 66.04 0)
+    (property "Value" "10u" (id 1) (at 111.7662 63.5 0)
+      (effects (font (size 1.27 1.27)) (justify left))
+    )
+    (property "Footprint" "Capacitor_SMD:C_0603_1608Metric_Pad1.08x0.95mm_HandSolder" (id 2) (at 110.49 66.04 0)
       (effects (font (size 1.27 1.27)) hide)
     )
@@
       (reference "#PWR040") (unit 1) (value "GND") (footprint "")
     )
-    (path "/8af304ee-0508-4120-992c-cb51500029d0/8d3e4c41-3045-4ea8-9a3f-316f92cb2b77"
-      (reference "#PWR041") (unit 1) (value "GND") (footprint "")
-    )
     (path "/8af304ee-0508-4120-992c-cb51500029d0/d0805c22-fe49-428f-b16a-1d51e7298a46"
       (reference "#PWR042") (unit 1) (value "GND") (footprint "")
     )
-    (path "/8af304ee-0508-4120-992c-cb51500029d0/4b8072e6-6935-4794-8ff0-3a6389d47708"
-      (reference "#PWR043") (unit 1) (value "GND") (footprint "")
-    )
     (path "/8af304ee-0508-4120-992c-cb51500029d0/4b180a30-f493-4e7b-949e-2cae4b349bbb"
       (reference "#PWR045") (unit 1) (value "+3.3V") (footprint "")
@@
       (reference "#PWR047") (unit 1) (value "+3.3VA") (footprint "")
     )
-    (path "/8af304ee-0508-4120-992c-cb51500029d0/eeb35366-9ed7-4ac3-ad67-f68724680744"
-      (reference "#PWR048") (unit 1) (value "GND") (footprint "")
-    )
     (path "/8af304ee-0508-4120-992c-cb51500029d0/0b01ec2a-61ec-4143-9d7d-6144b9de29b3"
       (reference "#PWR050") (unit 1) (value "GND") (footprint "")
     )
-    (path "/8af304ee-0508-4120-992c-cb51500029d0/f69faccb-d768-42ce-aacd-ceecd6cfc53a"
-      (reference "#PWR051") (unit 1) (value "GND") (footprint "")
-    )
     (path "/57827e05-5bc2-4fd8-89d5-a292512dab24/c6546110-a7b9-473a-83bd-e414d574c5e5"
       (reference "#PWR054") (unit 1) (value "GNDA") (footprint "")
@@
       (reference "#PWR0154") (unit 1) (value "GNDA") (footprint "")
     )
+    (path "/8af304ee-0508-4120-992c-cb51500029d0/0ca82de1-5d04-4582-af52-5412e4d49fa6"
+      (reference "#PWR0155") (unit 1) (value "GNDA") (footprint "")
+    )
+    (path "/8af304ee-0508-4120-992c-cb51500029d0/2cb296bb-04d8-4584-b85d-b6d6c7e76a9a"
+      (reference "#PWR0156") (unit 1) (value "GNDA") (footprint "")
+    )
+    (path "/8af304ee-0508-4120-992c-cb51500029d0/ebaad9b3-41e3-4c28-b683-f1bce292bc34"
+      (reference "#PWR0157") (unit 1) (value "GNDA") (footprint "")
+    )
+    (path "/8af304ee-0508-4120-992c-cb51500029d0/d8d4b2fc-8172-428e-ae35-ee5ee6797328"
+      (reference "#PWR0158") (unit 1) (value "GNDA") (footprint "")
+    )
     (path "/f0ee80f0-f258-4807-b18b-f799d7f64c1d/dd1bdb68-b5a4-43b3-ab1b-0af15c84ac32"

Commit message: routing
Connections:
- net CH1_D0: now also U3.37 (GPIO23); no longer U3.4 (SENSOR_VP/GPIO36/ADC1_CH0)
- net CH1_D1: now also U3.31 (GPIO19); no longer U3.5 (SENSOR_VN/GPIO39/ADC1_CH3)
- net CH1_D2: now also U3.30 (GPIO18); no longer U3.6 (GPIO34/ADC1_CH6)
- net CH1_D3: now also U3.29 (GPIO5); no longer U3.7 (GPIO35/ADC1_CH7)
- net CH1_D4: now also U3.28 (GPIO17); no longer U3.8 (32K_XP/GPIO32/ADC1_CH4)
- net CH1_D5: now also U3.27 (GPIO16); no longer U3.9 (32K_XN/GPIO33/ADC1_CH5)
- net CH1_D6: now also U3.26 (ADC2_CH0/GPIO4); no longer U3.13 (MTMS/GPIO14/ADC2_CH6)
- net CH1_D7: now also U3.24 (ADC2_CH2/GPIO2); no longer U3.14 (MTDI/GPIO12/ADC2_CH5)
- net CH2_D0: now also U3.4 (SENSOR_VP/GPIO36/ADC1_CH0); no longer U3.24 (ADC2_CH2/GPIO2)
- net CH2_D1: now also U3.5 (SENSOR_VN/GPIO39/ADC1_CH3); no longer U3.26 (ADC2_CH0/GPIO4)
- net CH2_D2: now also U3.6 (GPIO34/ADC1_CH6); no longer U3.29 (GPIO5)
- net CH2_D3: now also U3.7 (GPIO35/ADC1_CH7); no longer U3.27 (GPIO16)
- net CH2_D4: now also U3.8 (32K_XP/GPIO32/ADC1_CH4); no longer U3.28 (GPIO17)
- net CH2_D5: now also U3.9 (32K_XN/GPIO33/ADC1_CH5); no longer U3.30 (GPIO18)
- net CH2_D6: now also U3.13 (MTMS/GPIO14/ADC2_CH6); no longer U3.31 (GPIO19)
- net CH2_D7: now also U3.14 (MTDI/GPIO12/ADC2_CH5); no longer U3.37 (GPIO23)
- net GND: now also C10.2, C3.2, C9.2, IC2.1 (GND_1), IC2.29 (GND_5), IC2.32 (GND_6)
- net GNDREF: now also IC2.10 (~{AINB}), IC2.3 (~{AINA})
- removed net GNDA: C10.2, C3.2, C9.2, IC2.1 (GND_1), IC2.10 (~{AINB}), IC2.29 (GND_5), IC2.3 (~{AINA}), IC2.32 (GND_6)
- no-connect marks 4 -> 5
