File: _autosave-Analog.kicad_sch (KiCad schematic)
At the start: 37 parts

Commit message: layout for changed chematic
Connections:
- net GNDA: no longer D10.2 (A), D8.2 (A), IC6.4 (VSS), IC7.4 (VSS), IC8.2 (GND), IC9.2 (GND), U10.4 (V-), U8.4 (V-), U9.4 (V-)
- net SCL renamed SCL_I2C
- new net GND: D10.2 (A), D8.2 (A), IC6.4 (VSS), IC7.4 (VSS), IC8.2 (GND), IC9.2 (GND), U10.4 (V-), U8.4 (V-), U9.4 (V-)
