File: test.kicad_pcb (KiCad board)
At the start: 4 copper layers, 100 x 50 mm, 112 parts, among them IC1 USBLC6-2SC6, IC10 DAC5571IDBVR, IC2 ESP32-S3-WROOM-1-N16, IC3 MAX17048G+T10, IC4 BQ24074RGTR, IC5 LM4041CEM3-ADJ_NOPB, IC6 MCP6S91-E_MS, IC7 MCP6S91-E_MS, IC8 MCP4726A0T-E_CH, IC9 DAC5571IDBVR, J1 PWM, J2 UART0, K1 AQY210EHAX, K2 AQY210EHAX, SW1 Reset, SW2 Button, SW3 SW_DPDT_x2, U1 USB-TYPE-C-018, U10 MCP6022T-I_SN, U2 ADC08351CILQX/NOPB, U3 ADC08351CILQX/NOPB, U4 1043, U5 1043, U6 LD1086DT33TR, U7 LD1086DT33TR, U8 MCP6022T-I_SN, U9 MCP6022T-I_SN

Commit message: updated circuit
Parts:
- added C10: 0.1u, Capacitor_SMD:C_0603_1608Metric_Pad1.08x0.95mm_HandSolder, F.Cu at (191.5, 115.7)
- added C11: 0.1u, Capacitor_SMD:C_0603_1608Metric_Pad1.08x0.95mm_HandSolder, F.Cu at (181.7, 126.0)
- added C12: 0.1u, Capacitor_SMD:C_0603_1608Metric_Pad1.08x0.95mm_HandSolder, F.Cu at (165.5, 77.4)
- added C13: 0.1u, Capacitor_SMD:C_0603_1608Metric_Pad1.08x0.95mm_HandSolder, F.Cu at (198.8, 109.1)
- added C18: 0.1u, Capacitor_SMD:C_0805_2012Metric_Pad1.18x1.45mm_HandSolder, F.Cu at (198.8, 112.1)
- added C2: 0.1u, Capacitor_SMD:C_0603_1608Metric_Pad1.08x0.95mm_HandSolder, F.Cu at (172.8, 132.4)
- added C3: 0.1u, Capacitor_SMD:C_0603_1608Metric_Pad1.08x0.95mm_HandSolder, F.Cu at (172.8, 135.4)
- added C4: 0.1u, Capacitor_SMD:C_0805_2012Metric_Pad1.18x1.45mm_HandSolder, F.Cu at (177.6, 132.4)
- added C5: 0.1u, Capacitor_SMD:C_0603_1608Metric_Pad1.08x0.95mm_HandSolder, F.Cu at (184.3, 123.0)
- added C9: 0.1u, Capacitor_SMD:C_0603_1608Metric_Pad1.08x0.95mm_HandSolder, F.Cu at (154.1, 75.2)
- added D1: Status, LED_SMD:LED_0805_2012Metric_Pad1.15x1.40mm_HandSolder, F.Cu at (191.5, 118.8)
- added IC5: TCA9534APWR, project_library:SOP65P640X120-16N, F.Cu at (133.1, 67.6)
- added Q1: SS8050-G, project_library:SOT95P240X115-3N, F.Cu at (127.1, 73.5)
- added Q2: SS8050-G, project_library:SOT95P240X115-3N, F.Cu at (152.1, 137.6)
- added R15: 1k5, Resistor_SMD:R_0805_2012Metric_Pad1.20x1.40mm_HandSolder, F.Cu at (196.3, 115.7)
- added R16: 6k8, Resistor_SMD:R_0805_2012Metric_Pad1.20x1.40mm_HandSolder, F.Cu at (182.4, 131.9)
- added R17: 6k8, Resistor_SMD:R_0805_2012Metric_Pad1.20x1.40mm_HandSolder, F.Cu at (177.6, 135.4)
- added R3: 22.1k, Resistor_SMD:R_0805_2012Metric_Pad1.20x1.40mm_HandSolder, F.Cu at (181.6, 129.0)
- added R4: 47.5k, Resistor_SMD:R_0805_2012Metric_Pad1.20x1.40mm_HandSolder, F.Cu at (189.1, 123.0)
- added R5: 2k, Resistor_SMD:R_0805_2012Metric_Pad1.20x1.40mm_HandSolder, F.Cu at (186.4, 126.0)
- added R6: 10k, Resistor_SMD:R_0805_2012Metric_Pad1.20x1.40mm_HandSolder, F.Cu at (203.6, 109.0)
- added R7: 10k, Resistor_SMD:R_0805_2012Metric_Pad1.20x1.40mm_HandSolder, F.Cu at (171.3, 138.4)
- added R8: 10k, Resistor_SMD:R_0805_2012Metric_Pad1.20x1.40mm_HandSolder, F.Cu at (176.1, 138.4)
- added TP4: GNDREF, TestPoint:TestPoint_Keystone_5000-5004_Miniature, F.Cu at (196.4, 78.4)
- C6: value 1u -> 0.1u
- IC2: value ESP32-S3-WROOM-1-N16 -> AD9288BSTZ-40; footprint project_library:ESP32-S3-WROOM-1 -> project_library:QFP50P900X900X160-48N-AD9288
- J1: moved to F.Cu
- TP10: value ? -> OFFCH2
- TP11: value ? -> TRIGREF
- TP5: value ~ -> ANICH1
- TP6: value ~ -> ANICH2
- TP7: value ~ -> ANOCH1
- TP8: value ~ -> ANOCH2
- TP9: value ? -> OFFCH1
- U2: value ADC08351CILQX/NOPB -> CP2102N-A02-GQFN28; footprint project_library:ADC08351CILQX -> Package_DFN_QFN:QFN-28-1EP_5x5mm_P0.5mm_EP3.35x3.35mm
- U3: value ADC08351CILQX/NOPB -> ESP32-WROOM-E; footprint project_library:ADC08351CILQX -> Espressif:ESP32-WROOM-32E
- moved U2 54.9 mm to (185.5, 117.8)
- moved U3 21.2 mm to (143.1, 84.3), turned to 180 degrees
- moved IC2 16.5 mm to (159.5, 82.4)
- moved SW2 0.10 mm to (106.0, 58.9)
Connections:
- C19 pad 1: Net-(C18-Pad1) -> Net-(C19-Pad1)
- C20 pad 1: Net-(C18-Pad1) -> Net-(C19-Pad1)
- IC2 pad 1: GND -> GNDA
- IC2 pad 10: /CH2_D1 -> unconnected-(IC2-Pad10)
- IC2 pad 11: /CH2_D0 -> Analog_Out_CH2
- IC2 pad 12: /I2S_CLK -> Net-(C12-Pad1)
- IC2 pad 13: /USB_D- -> Net-(C12-Pad2)
- IC2 pad 14: /USB_D+ -> /I2S_CLK
- IC2 pad 15: /CH1_D7 -> +3V3
- IC2 pad 16: unconnected-(IC2-Pad16) -> GND
- IC2 pad 17: /CH1_D6 -> /CH2_D7
- IC2 pad 18: /CH1_D5 -> /CH2_D6
- IC2 pad 19: MOSI -> /CH2_D5
- IC2 pad 2: +3V3 -> Analog_Out_CH1
- IC2 pad 20: SCLK_SPI -> /CH2_D4
- IC2 pad 21: /CH1_D4 -> /CH2_D3
- IC2 pad 22: /CH1_D3 -> /CH2_D2
- IC2 pad 23: /CH1_D2 -> /CH2_D1
- IC2 pad 24: /CH1_D1 -> /CH2_D0
- IC2 pad 25: /CH1_D0 -> unconnected-(IC2-Pad25)
- IC2 pad 27: Net-(IC2-Pad27) -> GND
- IC2 pad 28: /Status_PWM -> +3V3
- IC2 pad 29: Trigger_CH1 -> GNDA
- IC2 pad 3: /ENABLE -> unconnected-(IC2-Pad3)
- IC2 pad 30: Trigger_CH2 -> +3.3VA
- IC2 pad 31: SDA -> +3.3VA
- IC2 pad 32: SCL_I2C -> GNDA
- IC2 pad 33: CH1_AC_Sel -> +3V3
- IC2 pad 34: CS_Gain_CH1 -> GND
- IC2 pad 35: Charging -> unconnected-(IC2-Pad35)
- IC2 pad 36: /RX0 -> unconnected-(IC2-Pad36)
- IC2 pad 37: /TX0 -> /CH1_D0
- IC2 pad 38: CS_Gain_CH2 -> /CH1_D1
- IC2 pad 39: CH2_AC_Sel -> /CH1_D2
- IC2 pad 4: /CH2_D7 -> +3V3
- IC2 pad 40: GND -> /CH1_D3
- IC2 pad 41: GND -> /CH1_D4
- IC2 pad 5: /CH2_D6 -> GNDREF
- IC2 pad 6: /CH2_D5 -> GNDREF
- IC2 pad 7: /CH2_D4 -> GNDREF
- IC2 pad 8: /CH2_D3 -> +3V3
- IC2 pad 9: /CH2_D2 -> +3V3
- JP1 pad 2: Net-(C18-Pad1) -> Net-(C19-Pad1)
- SW2 pad A: Net-(IC2-Pad27) -> GND
- SW2 pad B: Net-(IC2-Pad27) -> GND
- SW2 pad C: GND -> /IO0
- SW2 pad D: GND -> /IO0
- TP10 pad 1: /Analog/Offset_CH2 -> Offset_CH2
- TP9 pad 1: /Analog/Offset_CH1 -> Offset_CH1
- U2 pad 1: /CH1_D0 -> unconnected-(U2-Pad1)
- U2 pad 11: /I2S_CLK -> Net-(R6-Pad1)
- U2 pad 12: +3V3 -> unconnected-(U2-Pad12)
- U2 pad 14: +3.3VA -> unconnected-(U2-Pad14)
- U2 pad 15: GND -> unconnected-(U2-Pad15)
- U2 pad 16: +3.3VA -> unconnected-(U2-Pad16)
- U2 pad 17: Analog_Out_CH1 -> unconnected-(U2-Pad17)
- U2 pad 18: GND -> unconnected-(U2-Pad18)
- U2 pad 19: GND -> unconnected-(U2-Pad19)
- U2 pad 2: /CH1_D1 -> unconnected-(U2-Pad2)
- U2 pad 21: GND -> unconnected-(U2-Pad21)
- U2 pad 22: GND -> unconnected-(U2-Pad22)
- U2 pad 23: GND -> unconnected-(U2-Pad23)
- U2 pad 24: unconnected-(U2-Pad24) -> /RTS
- U2 pad 25: GND -> /RX
- U2 pad 3: /CH1_D2 -> GND
- U2 pad 4: /CH1_D3 -> /USB_D+
- U2 pad 5: /CH1_D4 -> /USB_D-
- U2 pad 6: /CH1_D5 -> +3V3
- U2 pad 7: /CH1_D6 -> +3V3
- U2 pad 8: /CH1_D7 -> Net-(R3-Pad2)
- U2 pad 9: unconnected-(U2-Pad9) -> Net-(R5-Pad2)
- U3 pad 1: /CH2_D0 -> GND
- U3 pad 10: unconnected-(U3-Pad10) -> Offset_CH1
- U3 pad 11: /I2S_CLK -> Offset_CH2
- U3 pad 12: +3V3 -> /I2S_CLK
- U3 pad 13: unconnected-(U3-Pad13) -> SCLK_SPI
- U3 pad 14: +3.3VA -> /CH1_D1
- U3 pad 16: +3.3VA -> MOSI
- U3 pad 17: Analog_Out_CH2 -> unconnected-(U3-Pad17)
- U3 pad 18: GND -> unconnected-(U3-Pad18)
- U3 pad 19: GND -> unconnected-(U3-Pad19)
- U3 pad 2: /CH2_D1 -> +3V3
- U3 pad 21: GND -> unconnected-(U3-Pad21)
- U3 pad 22: GND -> unconnected-(U3-Pad22)
- U3 pad 23: GND -> /CH1_D0
- U3 pad 24: unconnected-(U3-Pad24) -> /CH2_D7
- U3 pad 25: GND -> /IO0
- U3 pad 3: /CH2_D2 -> /ENABLE
- U3 pad 4: /CH2_D3 -> /CH1_D7
- U3 pad 5: /CH2_D4 -> /CH1_D6
- U3 pad 6: /CH2_D5 -> /CH1_D5
- U3 pad 7: /CH2_D6 -> /CH1_D4
- U3 pad 8: /CH2_D7 -> /CH1_D3
- U3 pad 9: unconnected-(U3-Pad9) -> /CH1_D2
- U6 pad 3: Net-(C18-Pad1) -> Net-(C19-Pad1)
- U7 pad 3: Net-(C18-Pad1) -> Net-(C19-Pad1)
- U8 pad 5: /Analog/Offset_CH1 -> Offset_CH1
- U9 pad 5: /Analog/Offset_CH2 -> Offset_CH2
Routing:
- net GND: track 128.0 -> 0.00 mm, vias 5 -> 0
- net SCL_I2C: track 102.0 -> 0.00 mm, vias 4 -> 0
- net /Status_PWM: track 98.3 -> 0.00 mm, vias 2 -> 0
- net SDA: track 97.0 -> 0.00 mm, vias 3 -> 0
- net Net-(IC2-Pad27): track 87.9 -> 0.00 mm, vias 2 -> 0
- net Net-(C18-Pad1): track 79.0 -> 0.00 mm, vias 4 -> 0
- net +3V3: track 113.6 -> 40.0 mm, vias 6 -> 0
- net GNDREF: track 65.3 -> 0.00 mm
- net CH1_AC_Sel: track 64.5 -> 0.00 mm, vias 2 -> 0
- net Net-(C17-Pad1): track 64.2 -> 0.00 mm, vias 2 -> 0
- net /ENABLE: track 61.2 -> 0.00 mm, vias 2 -> 0
- net CH2_AC_Sel: track 61.1 -> 0.00 mm, vias 2 -> 0
- net /RX0: track 59.5 -> 0.00 mm, vias 2 -> 0
- net SCLK_SPI: track 58.8 -> 0.00 mm, vias 4 -> 0
- net /TX0: track 56.7 -> 0.00 mm, vias 2 -> 0
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
Commit message: routing
Parts:
- removed the C10 at (162.5, 73.3)
- removed the C10 at (191.5, 115.7)
- removed the C11 at (167.7, 68.8)
- removed the C11 at (181.7, 126.0)
- removed the C12 at (167.7, 70.8)
- removed the C12 at (165.5, 77.4)
- removed the C13 at (198.8, 109.1)
- removed the C13 at (167.7, 72.8)
- removed the C18 at (182.3, 71.8)
- removed the C18 at (198.8, 112.1)
- removed the C2 at (172.8, 132.4)
- removed the C2 at (164.5, 95.2)
- removed C23: 1u, Capacitor_SMD:C_0805_2012Metric_Pad1.18x1.45mm_HandSolder
- removed the C3 at (168.3, 94.0)
- removed the C3 at (172.8, 135.4)
- removed the C4 at (168.3, 92.0)
- removed the C4 at (177.6, 132.4)
- removed the C5 at (184.3, 123.0)
- removed the C5 at (168.3, 90.0)
- removed the C9 at (164.5, 73.3)
- removed the D1 at (191.5, 118.8)
- removed the D1 at (135.5, 52.5)
- removed IC10, IC9: DAC5571IDBVR, project_library:DAC5571IDBVR
- removed the IC5 at (133.1, 67.6)
- removed the IC5 at (187.3, 72.0)
- removed J2: UART0, Connector_PinHeader_2.54mm:PinHeader_1x04_P2.54mm_Vertical
- removed the R15 at (184.3, 70.0)
- removed the R15 at (196.3, 115.7)
- removed the R16 at (187.3, 69.0)
- removed the R16 at (182.4, 131.9)
- removed the R17 at (190.5, 71.8)
- removed the R17 at (177.6, 135.4)
- removed the R3 at (181.6, 129.0)
- removed the R3 at (106.8, 81.1)
- removed the R4 at (189.1, 123.0)
- removed the R4 at (129.9, 83.8)
- removed the R5 at (186.4, 126.0)
- removed the R5 at (131.0, 81.8)
- removed the R6 at (184.5, 90.5)
- removed the R6 at (203.6, 109.0)
- removed the R7 at (182.0, 90.5)
- removed the R7 at (171.3, 138.4)
- removed the R8 at (135.5, 56.5)
- removed the R8 at (176.1, 138.4)
- removed the TP4 at (195.8, 69.2)
- added C10: 0.1u, Capacitor_SMD:C_0603_1608Metric_Pad1.08x0.95mm_HandSolder, F.Cu at (122.4, 90.3)
- added C11: 0.1u, Capacitor_SMD:C_0603_1608Metric_Pad1.08x0.95mm_HandSolder, F.Cu at (125.8, 90.3)
- added C12: 0.1u, Capacitor_SMD:C_0603_1608Metric_Pad1.08x0.95mm_HandSolder, F.Cu at (115.4, 77.7)
- added C13: 0.1u, Capacitor_SMD:C_0603_1608Metric_Pad1.08x0.95mm_HandSolder, F.Cu at (114.5, 81.7)
- added C18: 10u, Capacitor_SMD:C_0603_1608Metric_Pad1.08x0.95mm_HandSolder, F.Cu at (115.4, 79.2)
- added C2: 0.1u, Capacitor_SMD:C_0603_1608Metric_Pad1.08x0.95mm_HandSolder, F.Cu at (126.8, 79.9)
- added C3: 0.1u, Capacitor_SMD:C_0603_1608Metric_Pad1.08x0.95mm_HandSolder, F.Cu at (124.7, 78.2)
- added C4: 0.1u, Capacitor_SMD:C_0603_1608Metric_Pad1.08x0.95mm_HandSolder, F.Cu at (103.5, 83.9)
- added C5: 0.1u, Capacitor_SMD:C_0603_1608Metric_Pad1.08x0.95mm_HandSolder, F.Cu at (115.6, 90.3)
- added D1: Status, LED_SMD:LED_0805_2012Metric_Pad1.15x1.40mm_HandSolder, F.Cu at (149.7, 51.2)
- added IC5: TCA9534APWR, project_library:SOP65P640X120-16N, F.Cu at (157.3, 62.8)
- added R15: 10k, Resistor_SMD:R_0603_1608Metric_Pad0.98x0.95mm_HandSolder, F.Cu at (129.7, 70.2)
- added R16: 6k8, Resistor_SMD:R_0805_2012Metric_Pad1.20x1.40mm_HandSolder, F.Cu at (139.7, 65.7)
- added R17: 6k8, Resistor_SMD:R_0805_2012Metric_Pad1.20x1.40mm_HandSolder, F.Cu at (137.6, 65.7)
- added R3: 22.1k, Resistor_SMD:R_0603_1608Metric_Pad0.98x0.95mm_HandSolder, F.Cu at (119.7, 67.1)
- added R4: 47.5k, Resistor_SMD:R_0603_1608Metric_Pad0.98x0.95mm_HandSolder, F.Cu at (119.7, 65.6)
- added R5: 2k, Resistor_SMD:R_0603_1608Metric_Pad0.98x0.95mm_HandSolder, F.Cu at (119.7, 68.7)
- added R6: 10k, Resistor_SMD:R_0603_1608Metric_Pad0.98x0.95mm_HandSolder, F.Cu at (119.7, 70.2)
- added R7: 1k5, Resistor_SMD:R_0805_2012Metric_Pad1.20x1.40mm_HandSolder, F.Cu at (149.7, 55.0)
- added R8: 10k, Resistor_SMD:R_0603_1608Metric_Pad0.98x0.95mm_HandSolder, F.Cu at (129.7, 66.6)
- C1, C14, C15, C16, C17, C30, C31, C32, C6, C7, C8: footprint Capacitor_SMD:C_0805_2012Metric_Pad1.18x1.45mm_HandSolder -> Capacitor_SMD:C_0603_1608Metric_Pad1.08x0.95mm_HandSolder
- J1: moved to B.Cu
- R1, R10, R11, R2, R9: footprint Resistor_SMD:R_0805_2012Metric_Pad1.20x1.40mm_HandSolder -> Resistor_SMD:R_0603_1608Metric_Pad0.98x0.95mm_HandSolder
- R22, R23: value 835k -> 900k
- R24, R25: value 165k -> 100k
- moved U2 78.8 mm to (124.6, 67.8), turned to -90 degrees
- moved Q2 74.3 mm to (133.3, 65.6)
- moved C1 49.6 mm to (124.0, 63.9), turned to 0 degrees
- moved TP10 40.2 mm to (174.2, 79.6)
- moved IC2 39.0 mm to (120.5, 83.5), turned to -90 degrees
- moved C9 38.2 mm to (119.0, 90.3), turned to 180 degrees
- moved C32 36.7 mm to (165.8, 90.5), turned to 90 degrees
- moved IC8 31.8 mm to (162.3, 90.2), turned to 180 degrees
- moved IC3 30.5 mm to (146.4, 60.8), turned to 90 degrees
- moved C16 30.2 mm to (146.4, 63.2), turned to 180 degrees
- moved C31 30.1 mm to (159.4, 85.2)
- moved R9 29.6 mm to (118.6, 58.6), turned to -90 degrees
- moved C30 28.0 mm to (157.8, 85.2)
- moved TP2 26.8 mm to (138.3, 52.9)
- moved R11 26.5 mm to (115.0, 58.6), turned to 90 degrees
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Connections:
- net /DTR renamed /USB and GPIO Expander/DTR
- net /RTS renamed /USB and GPIO Expander/RTS
- net /USB_D+ renamed Net-(IC1-Pad3)
- net /USB_D- renamed Net-(IC1-Pad1)
- C30 pad 2: GND -> GNDA
- C31 pad 2: GND -> GNDA
- C32 pad 2: GND -> GNDA
- C6 pad 1: /ENABLE -> IO0
- D10 pad 2: GND -> GNDA
- D8 pad 2: GND -> GNDA
- IC2 pad 10: unconnected-(IC2-Pad10) -> GNDA
- IC2 pad 3: unconnected-(IC2-Pad3) -> GNDA
- IC6 pad 4: GND -> GNDA
- IC7 pad 4: GND -> GNDA
- IC8 pad 2: GND -> GNDA
- J1 pad 1: /Status_PWM -> /USB and GPIO Expander/Status_PWM
- Q1 pad 3: /ENABLE -> ENABLE
- Q2 pad 3: /IO0 -> IO0
- SW1 pad C: /ENABLE -> ENABLE
- SW1 pad D: /ENABLE -> ENABLE
- SW2 pad C: /IO0 -> IO0
- SW2 pad D: /IO0 -> IO0
- U10 pad 4: GND -> GNDA
- U2 pad 25: /RX -> /USB and GPIO Expander/RX
- U2 pad 26: /TX -> /USB and GPIO Expander/TX
- U3 pad 13: SCLK_SPI -> /CH1_D6
- U3 pad 14: /CH1_D1 -> /CH1_D7
- U3 pad 16: MOSI -> Trigger_CH2
- U3 pad 23: /CH1_D0 -> Trigger_CH1
- U3 pad 24: /CH2_D7 -> /CH2_D0
- U3 pad 26: /CH2_D6 -> /CH2_D1
- U3 pad 27: /CH2_D4 -> /CH2_D3
- U3 pad 28: /CH2_D3 -> /CH2_D4
- U3 pad 29: /CH2_D5 -> /CH2_D2
- U3 pad 30: /CH2_D2 -> /CH2_D5
- U3 pad 31: /CH2_D1 -> /CH2_D6
- U3 pad 37: /CH2_D0 -> /CH2_D7
- U3 pad 4: /CH1_D7 -> /CH1_D0
- U3 pad 5: /CH1_D6 -> /CH1_D1
- U3 pad 6: /CH1_D5 -> /CH1_D2
- U3 pad 7: /CH1_D4 -> /CH1_D3
- U3 pad 8: /CH1_D3 -> /CH1_D4
- U3 pad 9: /CH1_D2 -> /CH1_D5
- U8 pad 4: GND -> GNDA
- U9 pad 4: GND -> GNDA
Routing:
- net GNDREF: track 0.00 -> 68.6 mm
- net GND: track 0.00 -> 65.7 mm
- net /USB and GPIO Expander/Status_PWM: track 0.00 -> 58.7 mm, vias 0 -> 1
- net +3V3: track 40.0 -> 78.7 mm, vias 0 -> 1
- net Net-(C27-Pad1): track 0.00 -> 31.3 mm
- net CH1_AC_Sel: track 0.00 -> 27.9 mm, vias 0 -> 2
- net Net-(C26-Pad1): track 0.00 -> 27.5 mm
- net +3.3VA: track 0.00 -> 26.6 mm, vias 0 -> 4
- net Net-(IC7-Pad2): track 0.00 -> 23.0 mm
- net GNDA: track 0.00 -> 19.3 mm, vias 0 -> 4
- net Net-(IC6-Pad2): track 0.00 -> 14.9 mm
- net Analog_Out_CH2: track 0.00 -> 13.1 mm
- net Net-(J3-Pad3): track 0.00 -> 12.6 mm
- net Net-(C25-Pad1): track 0.00 -> 11.1 mm
- net Net-(Q2-Pad1): track 0.00 -> 9.58 mm
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
Commit message: routing
Parts:
- moved SW3 109.3 mm to (217.3, 36.9), turned to 0 degrees
- moved JP1 44.9 mm to (108.2, 51.1)
- moved TP11 40.1 mm to (174.2, 74.2)
- moved C2 32.4 mm to (158.6, 74.0)
- moved C10 32.4 mm to (154.2, 84.4)
- moved C11 32.4 mm to (157.6, 84.4)
- moved C12 32.4 mm to (147.2, 71.7)
- moved C18 32.4 mm to (147.2, 73.3)
- moved C3 32.4 mm to (156.5, 72.2)
- moved C5 32.4 mm to (147.4, 84.3)
- moved C9 32.4 mm to (150.8, 84.4)
- moved IC2 32.4 mm to (152.3, 77.5)
- moved C13 32.4 mm to (146.3, 75.7)
- moved U3 10.1 mm to (133.0, 84.3)
- moved C7 9.55 mm to (144.3, 90.3)
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Connections:
- C20 pad 2: GND -> GNDA
- C22 pad 2: GND -> GNDA
- D6 pad 1: GND -> GNDA
- U2 pad 25: /USB and GPIO Expander/RX -> RX
- U2 pad 26: /USB and GPIO Expander/TX -> TX
- U3 pad 25: /IO0 -> IO0
- U3 pad 3: /ENABLE -> ENABLE
- U3 pad 34: /RX -> RX
- U3 pad 35: /TX -> TX
- U7 pad 1: GND -> GNDA
Routing:
- net ENABLE: track 1.97 -> 67.0 mm
- net CH2_AC_Sel: track 0.00 -> 58.0 mm, vias 0 -> 2
- net GND: track 65.7 -> 114.2 mm
- net SDA: track 0.00 -> 45.6 mm
- net SCL_I2C: track 0.00 -> 45.6 mm
- net MOSI: track 0.00 -> 32.7 mm
- net SCLK_SPI: track 0.00 -> 29.3 mm
- net CS_Gain_CH2: track 0.00 -> 29.2 mm, vias 0 -> 2
- net /Power Supply/VBat+: track 0.00 -> 27.9 mm, vias 0 -> 2
- net GNDA: track 19.3 -> 45.7 mm, vias 4 -> 10
- net +3.3VA: track 26.6 -> 52.6 mm, vias 4 -> 8
- net +3V3: track 78.7 -> 101.9 mm, vias 1 -> 2
- net Charging: track 0.00 -> 21.6 mm
- net /I2S_CLK: track 0.00 -> 17.2 mm, vias 0 -> 2
- net +5V: track 0.00 -> 16.2 mm
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Other:
- outline, holes or cut-outs redrawn
